Commit message: aug 25

File: urdf/base.urdf (robot description, URDF)
Before this commit: robot mycobot_sim_base, 8 links, 7 joints
Joints:
- joint wheel_drive_L_joint: origin xyz=-0.345 -0.345 -0.07500000000000001 rpy=1.5708 0 0 -> xyz=-0.345 0.345 -0.07500000000000001 rpy=1.5708 0 0
- joint wheel_drive_R_joint: origin xyz=-0.345 0.345 -0.07500000000000001 rpy=1.5708 0 0 -> xyz=-0.345 -0.345 -0.07500000000000001 rpy=1.5708 0 0
- joint wheel_free_L_fork_joint: origin xyz=0.345 -0.345 -0.07500000000000001 rpy=0 0 0 -> xyz=0.345 0.345 -0.07500000000000001 rpy=0 0 0
- joint wheel_free_L_joint: origin xyz=0 0 0 rpy=1.5708 0 0 -> xyz=-0.06 0 0 rpy=1.5708 0 0
- joint wheel_free_R_fork_joint: origin xyz=0.345 0.345 -0.07500000000000001 rpy=0 0 0 -> xyz=0.345 -0.345 -0.07500000000000001 rpy=0 0 0
- joint wheel_free_R_joint: origin xyz=0 0 0 rpy=1.5708 0 0 -> xyz=-0.06 0 0 rpy=1.5708 0 0
